File: pa_23cm/current_sense.sch (EAGLE design)
At the start: 12 parts, among them IC1 MAX488CSA, IC2 7812T, IC3 7805T, J1 1X2-3.5MM

Commit message: working on current sensor board.  End of day commit.
Parts:
- removed FEATHER_32U4: FEATHERWING_NODIM, adafruit:FEATHERWING_NODIM
- removed H1, H2, H3, H4: MOUNT-HOLE5.5, holes:MOUNT-HOLE5.5
- removed IC2: 7812T, adafruit:7812T
- removed IC3: 7805T, adafruit:7805T
- removed J1: 1X2-3.5MM, adafruit:1X2-3.5MM
- added R2: 0, resistor:R-US_R0805
- IC1: value MAX488CSA -> INA250; device maxim:MAX488CSA -> vtgs:INA250
- R1: value 1k -> 0
- U$1: value DF13-5P-1.25H -> DF13-4P-1.25V; device con-hirose-df13:DF13-5P-1.25H -> con-hirose-df13:DF13-4P-1.25V
Connections:
- removed net +12V: IC1P.VCC
- removed net N$2: IC1G$1.B, R1.1
- removed net N$3: ADC1.SCL, FEATHER_32U4.GPIOSCL
- removed net N$8: ADC1.AIN3, U$1.4
- removed net N$9: IC2.VI, J1.2
- removed net RXD: FEATHER_32U4.GPIORX, IC1G$1.RO
- removed net TXD: FEATHER_32U4.GPIOTX, IC1G$1.DI
- new net SCL: ADC1.SCL, U$1.3
- new net SDA: ADC1.SDA, U$1.2
- new net V+: IC1.IN+@1, IC1.IN+@2, IC1.IN+@3
- new net V-: IC1.IN-@1, IC1.IN-@2, IC1.IN-@3
- net +3V3: now also IC1.VS, U$1.1
- net GND: now also IC1.GND@1, IC1.GND@2, IC1.GND@3, U$1.4; no longer IC1P.GND, J1.1, U$1.5
- net N$1: now also ADC1.AIN0, IC1.OUT; no longer IC1G$1.A, R1.2
- net N$4: now also IC1.SH-, R2.2; no longer ADC1.SDA, FEATHER_32U4.GPIOSDA
- net N$5: now also IC1.VIN-, R2.1; no longer ADC1.AIN0, U$1.1
- net N$6: now also IC1.SH+, R1.1; no longer ADC1.AIN1, U$1.2
- net N$7: now also IC1.VIN+, R1.2; no longer ADC1.AIN2, U$1.3
Other:
- moved on the sheet: ADC1, R1
