File: pa_vhf_uhf/temp_sensor/rev-/temp_sensor.sch (EAGLE design)
At the start: 0 parts

Commit message: final version of rev- for MCP9700 temp sensor for PA.
Parts:
- added C1: .1uF, rcl:C-USC0805K
- added IC1: MCP9700, vtgs:MCP9700
- added JP1: (no value), pinhead:PINHD-1X3
Connections:
- new net GND: C1.2, IC1.GND, JP1.1
- new net THERM: IC1.NC@1, IC1.NC@5
- new net VDD: C1.1, IC1.VDD, JP1.2
- new net VOUT: IC1.VOUT, JP1.3
